Commit message: Added and calibrated realsense camera. Must set realsense_link as the sensor frame in handeye gui.

File: irb120_control/urdf/irb120_3_58_macro.xacro (robot description, xacro)
@@ -219,5 +219,5 @@
     <link name="${prefix}tool0" />
     <joint name="${prefix}link_6-tool0" type="fixed">
-      <origin xyz="0 0 0" rpy="0 ${radians(90)} 0" />
+      <origin xyz="0 0 0" rpy="0 0 0" /> <!-- Was 0 90 0-->
       <parent link="${prefix}flange" />
       <child link="${prefix}tool0" />

File: irb120_control/urdf/irb120_with_finger.xacro (robot description, xacro)
@@ -38,8 +38,53 @@
   <xacro:property name="ft_length" value="0.08225"/>         <!-- FT sensor length -->
   <xacro:property name="finger_mass" value="0.066"/>      <!-- kg (finger) (from onshape) -->
-  <xacro:property name="finger_length" value="0.110"/>   <!-- finger length (from onshape)-->
+  <xacro:property name="finger_length" value="0.100"/>   <!-- finger length (from onshape)-->
+  <xacro:property name="finger_mesh" value="package://irb120_control/urdf/pusher_link.stl"/>
   <!-- Total offset from link_6 to finger tip will be ft_length + finger_length -->
-  <!-- Calibrated so that when finger_tip touches the table, FK reports z=-0.01199 in base_link -->
-  <xacro:property name="table_to_base_z" value="0.035"/>  <!-- was 0.01199 meters -->
+  <xacro:property name="table_thickness" value="0.044"/>
+  <xacro:property name="bracket_thickness" value="0.021"/>
+  <xacro:property name="table_center_x" value="0.40"/>
+  <xacro:property name="table_center_y" value="0.0"/>
+  <!-- FT sensor internal-frame mapping relative to link_6 (requested):
+       x_link6 ~ z_ft, y_link6 ~ -x_ft, z_link6 ~ -y_ft (right-hand completion).
+       Then we apply the inverse on ft_to_finger so finger stays in link_6/world-like
+       orientation at home for task reasoning. -->
+  <xacro:property name="ft_mount_roll" value="-1.5708"/>
+  <xacro:property name="ft_mount_pitch" value="0.0"/>
+  <xacro:property name="ft_mount_yaw" value="-1.5708"/>
+  <xacro:property name="finger_unwind_roll" value="0.0"/>
+  <xacro:property name="finger_unwind_pitch" value="-1.5708"/>
+  <xacro:property name="finger_unwind_yaw" value="1.5708"/>
+  <!-- world: base_link is at x=y=0; table top surface is z=0 -->
+  <link name="world"/>
+  <!-- ====== Table that the robot and object rest on (for collision and visuals) ====== -->
+  <link name='table'>
+    <visual>
+      <origin xyz="0 0 -${table_thickness / 2}" rpy="0 0 0"/>
+      <geometry>
+        <box size="2.0 0.8 ${table_thickness}"/>
+      </geometry>
+      <material name="Brown">
+        <color rgba="0.992 0.984 0.831 1.0"/>
+      </material>
+    </visual>
+    <collision>
+      <origin xyz="0 0 -${table_thickness / 2}" rpy="0 0 0"/>
+      <geometry>
+        <box size="2.0 0.8 ${table_thickness}"/>
+      </geometry>
+    </collision>
+  </link>
+  <!-- ====== Bracket that robot sits on, ontop of the table ====== -->
+  <link name='bracket'>
+    <visual>
+      <origin xyz="0 0 ${bracket_thickness / 2}" rpy="0 0 0"/>
+      <geometry>
+        <box size="0.194 0.8 ${bracket_thickness}"/>
+      </geometry>
+      <material name="LightGrey">
+        <color rgba="0.8 0.8 0.8 1.0"/>
+      </material>
+    </visual>
+  </link>
   <!-- ====== FT sensor link mounted to link_6 ====== -->
   <link name="ft_link">
@@ -54,73 +99,75 @@
         <cylinder radius="0.025" length="${ft_length}"/>
       </geometry>
-      <material name="Grey">
-        <color rgba="0.6 0.6 0.6 1.0"/>
+      <material name="LightGrey">
+        <color rgba="0.8 0.8 0.8 1.0"/>
       </material>
     </visual>
-    <!-- Basic cylinder collision geom -->
     <collision>
         <origin xyz="0 0 ${ft_length / 2}" rpy="0 0 0"/>
         <geometry>
-            <cylinder radius="0.025" length="${ft_length / 2.5}"/>
+            <cylinder radius="0.025" length="${ft_length / 2.5}"/> <!-- collision smaller to not interfere with finger (they never collide) -->
         </geometry>
     </collision>
   </link>
-  <joint name="link_6_to_ft" type="fixed">
-    <parent link="link_6"/>
-    <!-- Adjust xyz/rpy to match your real mounting orientation -->
-    <origin xyz="0 0 0" rpy="0 1.5708 0"/> <!-- Was 0.0001 0 0-->
-    <child link="ft_link"/>
-  </joint>
   <!-- ====== Finger link ====== -->
   <link name="finger_link">
-    <!-- Inertial properties -->
     <inertial>
-        <origin xyz="0 0 0.026" rpy="0 0 0"/>   <!-- adjust CoG -->
+        <origin xyz="0 0 0.026" rpy="0 1.5708 0"/>   <!-- adjust CoG -->
         <mass value="${finger_mass}"/>                   <!-- kg -->
         <inertia ixx="70.297" iyy="70.297" izz="70.297" ixy="0" ixz="0" iyz="0"/> <!-- kg mm^2-->
     </inertial>
-    <!-- Visual geometry -->
     <visual>
-      <origin xyz="0 0 ${finger_length / 2}" rpy="0 0 0"/>
+      <origin xyz="0 0 0" rpy="0 1.5708 0"/>
         <geometry>
-        <cylinder radius="0.008" length="${finger_length}"/>
+          <mesh filename="${finger_mesh}"/>
         </geometry>
-        <material name="white">
+        <material name="White">
             <color rgba="1.0 1.0 1.0 1.0"/>
         </material>
     </visual>
-    <!-- Simple cylinder geom -->
     <collision>
-        <origin xyz="0 0 ${finger_length / 4}" rpy="0 0 0"/>      <!-- adjust offset/orientation if needed -->
+        <origin xyz="0 0 0" rpy="0 1.5708 0"/>
         <geometry>
-            <cylinder radius=".008" length="${finger_length / 2}"/>
+            <mesh filename="${finger_mesh}"/>
         </geometry>
     </collision>
   </link>
+  <!-- ==================================== JOINTS ==================================== -->
+  <!-- connect link_6 to ft_link -->
+  <joint name="link_6_to_ft" type="fixed">
+    <parent link="link_6"/>
+    <origin
+      xyz="0 0 0"
+      rpy="${ft_mount_roll} ${ft_mount_pitch} ${ft_mount_yaw}"/>
+    <child link="ft_link"/>
+  </joint>
+  <!-- connect ft_link to finger_link -->
   <joint name="ft_to_finger" type="fixed">
     <parent link="ft_link"/>
-    <origin xyz="0 0 ${ft_length}" rpy="0 0 0"/> <!-- adjust as needed -->
+    <origin
+      xyz="0 0 ${ft_length}"
+      rpy="${finger_unwind_roll} ${finger_unwind_pitch} ${finger_unwind_yaw}"/>
     <child link="finger_link"/>
   </joint>
-  <!-- ====== Convenience EE frames ====== -->
-  <!-- tool0 at end of adapter (beginning of finger) -->
-  <!-- <link name="tool0"/>
-  <joint name="finger_adapter_to_tool0" type="fixed">
-    <parent link="finger_adapter"/>
-    <origin xyz="0 0 0" rpy="0 0 0"/>
-    <child link="tool0"/>
-  </joint> -->
-  <!-- finger_tip at the very end of the finger -->
-  <link name="finger_tip"/>
+  <!-- finger_ball_center at the very end of the finger for EE position (like mujoco 'site') -->
+  <link name="finger_ball_center"/>
   <joint name="finger_to_tip" type="fixed">
     <parent link="finger_link"/>
-    <origin xyz="0 0 ${finger_length}" rpy="0 0 0"/>
-    <child link="finger_tip"/>
+    <origin xyz="${finger_length} 0 0" rpy="0 0 0"/>
+    <child link="finger_ball_center"/>
   </joint>
-  <link name='table'/>
-  <!-- Table is the parent (world-ish), base_link is lifted above it by table_to_base_z -->
-  <joint name="table_to_base_link" type="fixed">
-    <parent link="table"/>
-    <origin xyz="0 0 ${table_to_base_z}" rpy="0 0 0"/>
+  <joint name="world_to_table" type="fixed">
+    <parent link="world"/>
+    <origin xyz="${table_center_x} ${table_center_y} 0" rpy="0 0 0"/>
+    <child link="table"/>
+  </joint>
+  <joint name="world_to_bracket" type="fixed">
+    <parent link="world"/>
+    <origin xyz="0 0 0" rpy="0 0 0"/>
+    <child link="bracket"/>
+  </joint>
+  <joint name="world_to_base" type="fixed">
+    <parent link="world"/>
+    <origin xyz="0 0 ${bracket_thickness}" rpy="0 0 0"/>
     <child link="base_link"/>
   </joint>

File: irb120_moveit_config/config/irb120_handeye_macro.srdf.xacro (robot description, xacro)
@@ -1,7 +1,7 @@
 <?xml version="1.0" encoding="utf-8"?>
 <robot xmlns:xacro="http://wiki.ros.org/xacro">
-  <xacro:macro name="irb120_srdf">
+  <xacro:macro name="irb120_handeye_srdf">
     <group name="manipulator">
-      <chain base_link="base_link" tip_link="finger_ball_center"/>
+      <chain base_link="base_link" tip_link="tool0"/>
     </group>
     <group_state name="all_zero" group="manipulator">
