Commit message: feat: Enhance DBSCAN SAM Culler with Depth Topic Support
- Added depth topic parameter to DBSCANSAMCuller for improved depth data handling.
- Implemented depth message subscription and processing alongside color messages.
- Updated metadata publishing to include depth information and its timestamp.
- Enhanced diagnostic capabilities by pairing depth data with RGB input for better analysis.

feat: Improve Pivot Boundary Review with Enhanced Press Comparison

- Integrated contact point selection into pivot boundary review for better decision-making.
- Updated review overlay to visualize both cloud and SAM pivot press points.
- Enhanced reporting to include detailed press comparison results and final choice validation.

fix: Refine Press Review Logic and Cleanup

- Removed unnecessary geometry rendering in press review.
- Ensured only the final queue of images is retained during review to optimize storage.

test: Add Comprehensive Tests for New Features

- Implemented tests for depth pairing in SAM diagnostics to ensure accurate timestamping.
- Added tests for approach diagnostics to validate position error calculations and FK usage.
- Created tests for cable limits to ensure trajectory validation works as expected.
- Developed tests for press targets to confirm correct behavior in RViz and motion planning contexts.

feat: Introduce Approach Diagnostics and Press Preview Utilities

- Added ApproachDiagnostics class for capturing and logging approach evidence.
- Implemented press preview functionality for visualizing saved snapshots in RViz.
- Created utility functions for managing press targets and building visualization markers.

File: irb120_control/urdf/irb120_3_58_macro.xacro (robot description, xacro)
@@ -197,5 +197,5 @@
       <parent link="${prefix}link_5"/>
       <child link="${prefix}link_6"/>
-      <limit effort="0" lower="-6.98132" upper="6.98132" velocity="7.33038"/>
+      <limit effort="0" lower="-1.0471975511965976" upper="1.0471975511965976" velocity="7.33038"/>
       <axis xyz="1 0 0"/>
       <dynamics damping="0.0" friction="0.0"/>
