Commit message: Added some object detection, two methods. 1) DBSCAN for density clustering from pointcloud, 2) SAM-2 with tiny weights for high-frequency runtime.

File: irb120_control/urdf/irb120_with_finger.xacro (robot description, xacro)
@@ -64,6 +64,6 @@
         <box size="2.0 0.8 ${table_thickness}"/>
       </geometry>
-      <material name="Brown">
-        <color rgba="0.992 0.984 0.831 1.0"/>
+      <material name="TableLight">
+        <color rgba="0.965 0.965 0.945 1.0"/>
       </material>
     </visual>

Commit message: Refactor IRB120 launch and control scripts
- Updated `bringup_irb120_moveit.launch.py` to streamline launch process and add preflight cleanup script.
- Introduced `ForceWatcher` class to monitor force and trigger actions based on contact detection.
- Added `netft_preprocessor.py` for filtering and reorienting NetFT wrench data.
- Implemented `squash_pull.py` for a Cartesian force control strategy during object manipulation.
- Created `preflight_cleanup.sh` script to handle cleanup of stale processes and reset USB devices before launching.
- Enhanced URDF definitions for collision detection and joint connections.
- Updated `setup.py` to include new scripts and entry points.

File: irb120_control/urdf/irb120_with_finger.xacro (robot description, xacro)
@@ -86,4 +86,10 @@
       </material>
     </visual>
+    <collision>
+      <origin xyz="0 0 ${bracket_thickness / 2}" rpy="0 0 0"/>
+      <geometry>
+        <box size="0.194 0.8 ${bracket_thickness}"/>
+      </geometry>
+    </collision>
   </link>
   <!-- ====== FT sensor link mounted to link_6 ====== -->
@@ -134,7 +140,7 @@
   </link>
   <!-- ==================================== JOINTS ==================================== -->
-  <!-- connect link_6 to ft_link -->
-  <joint name="link_6_to_ft" type="fixed">
-    <parent link="link_6"/>
+  <!-- connect tool0 to ft_link -->
+  <joint name="tool0_to_ft" type="fixed">
+    <parent link="tool0"/>
     <origin
       xyz="0 0 0"

Commit message: Added calibration for ft after noticing phantom weight under no finger load. Need to add description to README.

File: irb120_control/urdf/irb120_with_finger.xacro (robot description, xacro)
@@ -34,14 +34,18 @@
     configure_via_rws="${configure_via_rws}"/>
   <!-- ====== Params to tweak ====== -->
-  <xacro:property name="ft_mass" value="0.255"/>          <!-- kg (sensor) (from spec sheet) -->
-  <xacro:property name="ft_cog_z" value="0.063"/>         <!-- meters in tool frame (from spec sheet)-->
-  <xacro:property name="ft_length" value="0.08225"/>         <!-- FT sensor length -->
-  <xacro:property name="finger_mass" value="0.066"/>      <!-- kg (finger) (from onshape) -->
-  <xacro:property name="finger_length" value="0.100"/>   <!-- finger length (from onshape)-->
+  <xacro:property name="ft_mass" value="0.255"/>               <!-- kg (sensor) (from spec sheet) -->
+  <xacro:property name="ft_cog" value="0.063"/>              <!-- meters in tool frame (from spec sheet)-->
+  <xacro:property name="ft_length" value="0.08225"/>           <!-- FT sensor length (measured) -->
+  <xacro:property name="finger_mass" value="0.066"/>           <!-- kg (measured finger+ball+screws) -->
+  <xacro:property name="finger_cog" value="0.0275"/>         <!-- meters in finger frame (measured) -->
+  <xacro:property name="finger_length" value="0.100"/>         <!-- finger length (measured)-->
+  <xacro:property name="finger_ball_radius" value="0.01312"/>  <!-- Ball radius (measured 26.25 mm diameter)-->
+  <xacro:property name="finger_contact" value="0.0875"/>     <!-- finger contact length (measured ball center from base)-->
   <xacro:property name="finger_mesh" value="package://irb120_control/urdf/pusher_link.stl"/>
   <!-- Total offset from link_6 to finger tip will be ft_length + finger_length -->
-  <xacro:property name="table_thickness" value="0.044"/>
+  <!-- Total offset from link_6 to contact point will be ft_length + finger_contact -->
+  <xacro:property name="table_thickness" value="0.044"/> <!-- Visual feature -->
   <xacro:property name="bracket_thickness" value="0.021"/>
-  <xacro:property name="table_center_x" value="0.40"/>
+  <xacro:property name="table_center_x" value="0.40"/> <!-- Mostly visual, maybe for workspace bounds -->
   <xacro:property name="table_center_y" value="0.0"/>
   <!-- FT sensor internal-frame mapping relative to link_6 (requested):
@@ -49,10 +53,10 @@
        Then we apply the inverse on ft_to_finger so finger stays in link_6/world-like
        orientation at home for task reasoning. -->
-  <xacro:property name="ft_mount_roll" value="-1.5708"/>
+  <!-- <xacro:property name="ft_mount_roll" value="-1.5708"/>
   <xacro:property name="ft_mount_pitch" value="0.0"/>
-  <xacro:property name="ft_mount_yaw" value="-1.5708"/>
-  <xacro:property name="finger_unwind_roll" value="0.0"/>
+  <xacro:property name="ft_mount_yaw" value="-1.5708"/> -->
+  <!-- <xacro:property name="finger_unwind_roll" value="0.0"/>
   <xacro:property name="finger_unwind_pitch" value="-1.5708"/>
-  <xacro:property name="finger_unwind_yaw" value="1.5708"/>
+  <xacro:property name="finger_unwind_yaw" value="1.5708"/> -->
   <!-- world: base_link is at x=y=0; table top surface is z=0 -->
   <link name="world"/>
@@ -69,5 +73,5 @@
     </visual>
     <collision>
-      <origin xyz="0 0 -${table_thickness / 2}" rpy="0 0 0"/>
+      <origin xyz="0 0 -${table_thickness / 2}" rpy="0 0 0"/> <!-- At the center, bottom of table-->
       <geometry>
         <box size="2.0 0.8 ${table_thickness}"/>
@@ -96,10 +100,10 @@
   <link name="ft_link">
     <inertial>
-      <origin xyz="0 0 ${ft_cog_z}" rpy="0 0 0"/>
+      <origin xyz="${ft_cog} 0 0" rpy="0 1.5708 0"/>
       <mass value="${ft_mass}"/>
       <inertia ixx="5e-4" iyy="5e-4" izz="5e-4" ixy="0" ixz="0" iyz="0"/>
     </inertial>
     <visual>
-      <origin xyz="0 0 ${ft_length / 2}" rpy="0 0 0"/>
+      <origin xyz="${ft_length / 2} 0 0" rpy="0 1.5708 0"/>
       <geometry>
         <cylinder radius="0.025" length="${ft_length}"/>
@@ -110,7 +114,7 @@
     </visual>
     <collision>
-        <origin xyz="0 0 ${ft_length / 2}" rpy="0 0 0"/>
+        <origin xyz="${ft_length / 2} 0 0" rpy="0 1.5708 0"/>
         <geometry>
-            <cylinder radius="0.025" length="${ft_length / 2.5}"/> <!-- collision smaller to not interfere with finger (they never collide) -->
+            <cylinder radius="0.025" length="${ft_length / 2.5}"/> <!-- smaller to avoid finger interference (no collision anyways) -->
         </geometry>
     </collision>
@@ -119,7 +123,7 @@
   <link name="finger_link">
     <inertial>
-        <origin xyz="0 0 0.026" rpy="0 1.5708 0"/>   <!-- adjust CoG -->
-        <mass value="${finger_mass}"/>                   <!-- kg -->
-        <inertia ixx="70.297" iyy="70.297" izz="70.297" ixy="0" ixz="0" iyz="0"/> <!-- kg mm^2-->
+        <origin xyz="${finger_cog} 0 0" rpy="0 1.5708 0"/>   <!-- Rotate for correct attachment and orientation -->
+        <mass value="${finger_mass}"/>
+        <inertia ixx="70.297" iyy="70.297" izz="70.297" ixy="0" ixz="0" iyz="0"/>
     </inertial>
     <visual>
@@ -145,5 +149,5 @@
     <origin
       xyz="0 0 0"
-      rpy="${ft_mount_roll} ${ft_mount_pitch} ${ft_mount_yaw}"/>
+      rpy="0 0 0"/> <!-- Now we re-orient the FT sensor internally (net ft settings configuration)-->
     <child link="ft_link"/>
   </joint>
@@ -152,15 +156,16 @@
     <parent link="ft_link"/>
     <origin
-      xyz="0 0 ${ft_length}"
-      rpy="${finger_unwind_roll} ${finger_unwind_pitch} ${finger_unwind_yaw}"/>
+      xyz="${ft_length} 0 0"
+      rpy="0 0 0"/>
     <child link="finger_link"/>
   </joint>
-  <!-- finger_ball_center at the very end of the finger for EE position (like mujoco 'site') -->
+  <!-- finger_ball_center at contact point for EE position (like mujoco 'site') -->
   <link name="finger_ball_center"/>
-  <joint name="finger_to_tip" type="fixed">
+  <joint name="finger_to_ball_center" type="fixed">
     <parent link="finger_link"/>
-    <origin xyz="${finger_length} 0 0" rpy="0 0 0"/>
+    <origin xyz="${finger_contact} 0 0" rpy="0 0 0"/>
     <child link="finger_ball_center"/>
   </joint>
+  <!-- World and table should coincide, at the top table surface -->
   <joint name="world_to_table" type="fixed">
     <parent link="world"/>
