Commit message: Added new models for adapter for accuracy. Changed object detection to accept two cameras with combined clouds.

File: irb120_control/urdf/irb120_with_finger.xacro (robot description, xacro)
@@ -34,6 +34,4 @@
     configure_via_rws="${configure_via_rws}"/>
   <!-- ====== Params to tweak ====== -->
-  <xacro:property name="ft_mass" value="0.255"/>               <!-- kg (sensor) (from spec sheet) -->
-  <xacro:property name="ft_cog" value="0.063"/>              <!-- meters in tool frame (from spec sheet)-->
   <xacro:property name="ft_length" value="0.08225"/>           <!-- FT sensor length (measured) -->
   <xacro:property name="finger_mass" value="0.066"/>           <!-- kg (measured finger+ball+screws) -->
@@ -49,14 +47,4 @@
   <xacro:property name="table_center_x" value="0.40"/> <!-- Mostly visual, maybe for workspace bounds -->
   <xacro:property name="table_center_y" value="0.0"/>
-  <!-- FT sensor internal-frame mapping relative to link_6 (requested):
-       x_link6 ~ z_ft, y_link6 ~ -x_ft, z_link6 ~ -y_ft (right-hand completion).
-       Then we apply the inverse on ft_to_finger so finger stays in link_6/world-like
-       orientation at home for task reasoning. -->
-  <!-- <xacro:property name="ft_mount_roll" value="-1.5708"/>
-  <xacro:property name="ft_mount_pitch" value="0.0"/>
-  <xacro:property name="ft_mount_yaw" value="-1.5708"/> -->
-  <!-- <xacro:property name="finger_unwind_roll" value="0.0"/>
-  <xacro:property name="finger_unwind_pitch" value="-1.5708"/>
-  <xacro:property name="finger_unwind_yaw" value="1.5708"/> -->
   <!-- world: base_link is at x=y=0; table top surface is z=0 -->
   <link name="world"/>
@@ -97,27 +85,20 @@
     </collision>
   </link>
-  <!-- ====== FT sensor link mounted to link_6 ====== -->
-  <link name="ft_link">
-    <inertial>
-      <origin xyz="${ft_cog} 0 0" rpy="0 1.5708 0"/>
-      <mass value="${ft_mass}"/>
-      <inertia ixx="5e-4" iyy="5e-4" izz="5e-4" ixy="0" ixz="0" iyz="0"/>
-    </inertial>
-    <visual>
-      <origin xyz="${ft_length / 2} 0 0" rpy="0 1.5708 0"/>
-      <geometry>
-        <cylinder radius="0.025" length="${ft_length}"/>
-      </geometry>
-      <material name="LightGrey">
-        <color rgba="0.8 0.8 0.8 1.0"/>
-      </material>
-    </visual>
-    <collision>
-        <origin xyz="${ft_length / 2} 0 0" rpy="0 1.5708 0"/>
-        <geometry>
-            <cylinder radius="0.025" length="${ft_length / 2.5}"/> <!-- smaller to avoid finger interference (no collision anyways) -->
-        </geometry>
-    </collision>
-  </link>
+  <!-- ====== FT sensor + adapter stack, mounted to tool0 ====== -->
+  <!-- Accurate geometry/mass/collision now comes from the Onshape CAD export below
+       (root -> adapter_robot -> adapter_sensor -> sensor_plate -> sensor_body),
+       replacing the old hand-measured stand-in cylinder.
+       ft_link itself stays a bare frame (no visual/collision/inertial — same pattern
+       as finger_ball_center below) pinned EXACTLY where it always was: coincident
+       with tool0 (tool0_to_ft is identity). Do not move it or give it mass/inertia —
+       netft_preprocessor.py, calibrate_ft_sensor.py, and estimation/tst.py all
+       hardcode "ft_link" as the wrench TF frame and assume this exact position
+       (see tst.py's docstring); moving it or double-counting its mass against the
+       new CAD links' own inertials would silently break their lever-arm math. -->
+  <link name="ft_link"/>
+  <!-- Onshape CAD export: located in irb120_control/urdf/sensor_and_adapter_assembly.
+       Grafted onto tool0 as its own branch (parallel to ft_link/finger_link above),
+       not merged into the ft_link/finger chain. -->
+  <xacro:include filename="$(find irb120_control)/urdf/sensor_and_adapter_assembly/sensor_and_adapter_assembly.urdf"/>
   <!-- ====== Finger link ====== -->
   <link name="finger_link">
@@ -151,4 +132,16 @@
       rpy="0 0 0"/> <!-- Now we re-orient the FT sensor internally (net ft settings configuration)-->
     <child link="ft_link"/>
+  </joint>
+  <!-- connect tool0 to the Onshape assembly's root mate connector.
+       Starting with identity: assumes the mate connector picked as "root" when
+       exporting from Onshape was oriented to match tool0's convention (Z out
+       along the approach direction). VERIFY VISUALLY IN RVIZ — if the assembly
+       renders rotated/flipped relative to the real sensor mounting, adjust this
+       joint's rpy (nothing else needs to change; ft_link/finger_link above are
+       on a separate branch and unaffected either way). -->
+  <joint name="tool0_to_root" type="fixed">
+    <parent link="tool0"/>
+    <origin xyz="0 0 0" rpy="0 0 0"/>
+    <child link="root"/>
   </joint>
   <!-- connect ft_link to finger_link -->

Commit message: Updated robot model to be much more realistic and accurate to the real world, including mounting brackets, finger body and ball geometries. Updated press-point selection to work across several objects.

File: irb120_control/urdf/irb120_with_finger.xacro (robot description, xacro)
@@ -34,17 +34,13 @@
     configure_via_rws="${configure_via_rws}"/>
   <!-- ====== Params to tweak ====== -->
-  <xacro:property name="ft_length" value="0.08225"/>           <!-- FT sensor length (measured) -->
+  <xacro:property name="ft_body_length_xyz" value="0 0 -0.02975"/>  <!-- Literallly just the sensor body length. Sensor body 'origin' is its robot-side face. -->
   <xacro:property name="finger_mass" value="0.066"/>           <!-- kg (measured finger+ball+screws) -->
   <xacro:property name="finger_cog" value="0.0275"/>         <!-- meters in finger frame (measured) -->
   <xacro:property name="finger_length" value="0.100"/>         <!-- finger length (measured)-->
-  <xacro:property name="finger_ball_radius" value="0.01312"/>  <!-- Ball radius (measured 26.25 mm diameter)-->
-  <xacro:property name="finger_contact" value="0.0875"/>     <!-- finger contact length (measured ball center from base)-->
-  <xacro:property name="finger_mesh" value="package://irb120_control/urdf/pusher_link.stl"/>
-  <!-- Total offset from link_6 to finger tip will be ft_length + finger_length -->
-  <!-- Total offset from link_6 to contact point will be ft_length + finger_contact -->
+  <xacro:property name="finger_ball_radius" value="0.01325"/>  <!-- Ball radius, matches finger_assembly.urdf ball link's CAD inertial/mesh offset exactly -->
+  <xacro:property name="finger_ball_center_xyz" value="0 0 0.0866512"/>     <!-- finger_assembly.urdf CAD chain, root_finger's local Z is the shaft axis: 0 (root_finger->pusher_body) + 0.0734012 (pusher_body->ball) + 0.01325 (ball mesh recenter) -->
   <xacro:property name="table_thickness" value="0.044"/> <!-- Visual feature -->
-  <xacro:property name="bracket_thickness" value="0.021"/>
-  <xacro:property name="table_center_x" value="0.40"/> <!-- Mostly visual, maybe for workspace bounds -->
-  <xacro:property name="table_center_y" value="0.0"/>
+  <xacro:property name="bracket_thickness" value="0.021"/> <!-- Visual feature -->
+  <xacro:property name="table_center_xyz" value="0.40 0 0"/> <!-- Visual feature -->
   <!-- world: base_link is at x=y=0; table top surface is z=0 -->
   <link name="world"/>
@@ -85,31 +81,18 @@
     </collision>
   </link>
-  <!-- ====== FT sensor + adapter stack, mounted to tool0 ====== -->
-  <!-- Accurate geometry/mass/collision now comes from the Onshape CAD export below
-       (root -> adapter_robot -> adapter_sensor -> sensor_plate -> sensor_body),
-       replacing the old hand-measured stand-in cylinder.
-       ft_link itself stays a bare frame (no visual/collision/inertial — same pattern
-       as finger_ball_center below) pinned EXACTLY where it always was: coincident
-       with tool0 (tool0_to_ft is identity). Do not move it or give it mass/inertia —
-       netft_preprocessor.py, calibrate_ft_sensor.py, and estimation/tst.py all
-       hardcode "ft_link" as the wrench TF frame and assume this exact position
-       (see tst.py's docstring); moving it or double-counting its mass against the
-       new CAD links' own inertials would silently break their lever-arm math. -->
-  <link name="ft_link"/>
-  <!-- Onshape CAD export: located in irb120_control/urdf/sensor_and_adapter_assembly.
-       Grafted onto tool0 as its own branch (parallel to ft_link/finger_link above),
-       not merged into the ft_link/finger chain. -->
-  <xacro:include filename="$(find irb120_control)/urdf/sensor_and_adapter_assembly/sensor_and_adapter_assembly.urdf"/>
+  <!-- ====== FT sensor + adapter stack, mounted to tool0 + finger and ball ====== -->
+  <xacro:include filename="$(find irb120_control)/urdf/sensor_and_adapter_assembly.urdf"/>
+  <xacro:include filename="$(find irb120_control)/urdf/finger_assembly.urdf"/>
   <!-- ====== Finger link ====== -->
-  <link name="finger_link">
+  <!-- <link name="finger_link">
     <inertial>
-        <origin xyz="${finger_cog} 0 0" rpy="0 1.5708 0"/>   <!-- Rotate for correct attachment and orientation -->
+        <origin xyz="${finger_cog} 0 0" rpy="0 ${pi/2} 0"/>
         <mass value="${finger_mass}"/>
         <inertia ixx="70.297" iyy="70.297" izz="70.297" ixy="0" ixz="0" iyz="0"/>
     </inertial>
     <visual>
-      <origin xyz="0 0 0" rpy="0 1.5708 0"/>
+      <origin xyz="0 0 0" rpy="0 ${pi/2} 0"/>
         <geometry>
-          <mesh filename="${finger_mesh}"/>
+          <mesh filename="package://irb120_control/meshes/pusher_link.stl"/>
         </geometry>
         <material name="White">
@@ -118,44 +101,28 @@
     </visual>
     <collision>
-        <origin xyz="0 0 0" rpy="0 1.5708 0"/>
+        <origin xyz="0 0 0" rpy="0 ${pi/2} 0"/>
         <geometry>
-            <mesh filename="${finger_mesh}"/>
+            <mesh filename="package://irb120_control/meshes/pusher_link.stl"/>
         </geometry>
     </collision>
-  </link>
+  </link> -->
   <!-- ==================================== JOINTS ==================================== -->
-  <!-- connect tool0 to ft_link -->
-  <joint name="tool0_to_ft" type="fixed">
+  <!-- connect tool0 to the Onshape assembly's root mate connector -->
+  <joint name="tool0_to_sensor_root" type="fixed">
     <parent link="tool0"/>
-    <origin
-      xyz="0 0 0"
-      rpy="0 0 0"/> <!-- Now we re-orient the FT sensor internally (net ft settings configuration)-->
-    <child link="ft_link"/>
+    <origin xyz="0 0 0" rpy="0 0 ${pi/2}"/>
+    <child link="root_sensor"/>
   </joint>
-  <!-- connect tool0 to the Onshape assembly's root mate connector.
-       Starting with identity: assumes the mate connector picked as "root" when
-       exporting from Onshape was oriented to match tool0's convention (Z out
-       along the approach direction). VERIFY VISUALLY IN RVIZ — if the assembly
-       renders rotated/flipped relative to the real sensor mounting, adjust this
-       joint's rpy (nothing else needs to change; ft_link/finger_link above are
-       on a separate branch and unaffected either way). -->
-  <joint name="tool0_to_root" type="fixed">
-    <parent link="tool0"/>
-    <origin xyz="0 0 0" rpy="0 0 0"/>
-    <child link="root"/>
+  <!-- connect sensor_body to finger_link (sensor body origin is its robot-side face) -->
+  <joint name="sensor_body_to_finger_root" type="fixed">
+    <parent link="sensor_body"/>
+    <origin xyz="${ft_body_length_xyz}" rpy="0 ${pi} 0"/> <!--0.3971356 ${pi/2} -1.1736581"-->
+    <child link="root_finger"/>
   </joint>
-  <!-- connect ft_link to finger_link -->
-  <joint name="ft_to_finger" type="fixed">
-    <parent link="ft_link"/>
-    <origin
-      xyz="${ft_length} 0 0"
-      rpy="0 0 0"/>
-    <child link="finger_link"/>
-  </joint>
-  <!-- finger_ball_center at contact point for EE position (like mujoco 'site') -->
+  <!-- finger_ball_center for EE pose (like mujoco 'site') -->
   <link name="finger_ball_center"/>
   <joint name="finger_to_ball_center" type="fixed">
-    <parent link="finger_link"/>
-    <origin xyz="${finger_contact} 0 0" rpy="0 0 0"/>
+    <parent link="root_finger"/>
+    <origin xyz="${finger_ball_center_xyz}" rpy="0 0 0"/>
     <child link="finger_ball_center"/>
   </joint>
@@ -163,5 +130,5 @@
   <joint name="world_to_table" type="fixed">
     <parent link="world"/>
-    <origin xyz="${table_center_x} ${table_center_y} 0" rpy="0 0 0"/>
+    <origin xyz="${table_center_xyz}" rpy="0 0 0"/>
     <child link="table"/>
   </joint>

File: irb120_control/urdf/sensor_and_adapter_assembly.urdf (robot description, URDF)
Before this commit: robot sensor_and_adapter_assembly, 5 links, 4 joints
Links:
- removed link root
- added link root_sensor
- link adapter_robot: geometry collision mesh filename=package://irb120_control/meshes/sensor_and_adapter_assembly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 scale=1 1 1; visual mesh filename=package://irb120_control/meshes/sensor_and_adapter_assembly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 scale=1 1 1
- link adapter_sensor: geometry collision mesh filename=package://irb120_control/meshes/sensor_and_adapter_assembly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 scale=1 1 1; visual mesh filename=package://irb120_control/meshes/sensor_and_adapter_assembly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 scale=1 1 1
- link sensor_body: geometry visual mesh filename=package://irb120_control/meshes/sensor_and_adapter_assembly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 scale=1 1 1
- link sensor_plate: geometry collision mesh filename=package://irb120_control/meshes/sensor_and_adapter_assembly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 scale=1 1 1; visual mesh filename=package://irb120_control/meshes/sensor_and_adapter_assembly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 scale=1 1 1
Joints:
- joint fastened_1: origin xyz=0 0 0 rpy=-1.5708 -0 3.14159 -> xyz=0 0 0 rpy=-1.5708 0 3.14159; parent root -> root_sensor
- joint fastened_2: origin xyz=0 2.88889e-34 0.01 rpy=3.14159 -0 0 -> xyz=0 0 0.01 rpy=3.14159 0 0
- joint fastened_3: origin xyz=6.55487e-18 1.0842e-19 -0.0215 rpy=0 -0 5.05364e-31 -> xyz=0 0 -0.0215 rpy=0 0 0
- joint fastened_4: origin xyz=4.7813e-05 -0.000464975 -0.021 rpy=0 -0 3.14159 -> xyz=0 0 -0.021 rpy=0 0 3.14159

File: irb120_moveit_config/config/irb120_macro.srdf.xacro (robot description, xacro)
@@ -25,6 +25,11 @@
     <disable_collisions link1="link_4" link2="link_6" reason="Never"/>
     <disable_collisions link1="link_5" link2="link_6" reason="Adjacent"/>
-    <disable_collisions link1="link_6" link2="ft_link" reason="Adjacent"/>
-    <disable_collisions link1="ft_link" link2="finger_link" reason="Adjacent"/>
+    <disable_collisions link1="link_5" link2="adapter_sensor" reason="Adjacent"/> <!-- Recall the adapter 'sticks into' the tool0 to be secure. This avoids collision.-->
+    <disable_collisions link1="link_6" link2="adapter_robot" reason="Adjacent"/>
+    <disable_collisions link1="link_6" link2="adapter_sensor" reason="Adjacent"/>
+    <disable_collisions link1="adapter_robot" link2="adapter_sensor" reason="Adjacent"/>
+    <disable_collisions link1="adapter_sensor" link2="sensor_plate" reason="Adjacent"/>
+    <disable_collisions link1="sensor_body" link2="pusher_body" reason="Adjacent"/>
+    <disable_collisions link1="pusher_body" link2="ball" reason="Adjacent"/>
   </xacro:macro>
 </robot>

Commit message: Updated urdf s.t. finger_ball_Center frame is oriented correctly as defined across entire control stack (x fwd, z up).

File: irb120_control/urdf/irb120_with_finger.xacro (robot description, xacro)
@@ -84,27 +84,4 @@
   <xacro:include filename="$(find irb120_control)/urdf/sensor_and_adapter_assembly.urdf"/>
   <xacro:include filename="$(find irb120_control)/urdf/finger_assembly.urdf"/>
-  <!-- ====== Finger link ====== -->
-  <!-- <link name="finger_link">
-    <inertial>
-        <origin xyz="${finger_cog} 0 0" rpy="0 ${pi/2} 0"/>
-        <mass value="${finger_mass}"/>
-        <inertia ixx="70.297" iyy="70.297" izz="70.297" ixy="0" ixz="0" iyz="0"/>
-    </inertial>
-    <visual>
-      <origin xyz="0 0 0" rpy="0 ${pi/2} 0"/>
-        <geometry>
-          <mesh filename="package://irb120_control/meshes/pusher_link.stl"/>
-        </geometry>
-        <material name="White">
-            <color rgba="1.0 1.0 1.0 1.0"/>
-        </material>
-    </visual>
-    <collision>
-        <origin xyz="0 0 0" rpy="0 ${pi/2} 0"/>
-        <geometry>
-            <mesh filename="package://irb120_control/meshes/pusher_link.stl"/>
-        </geometry>
-    </collision>
-  </link> -->
   <!-- ==================================== JOINTS ==================================== -->
   <!-- connect tool0 to the Onshape assembly's root mate connector -->
@@ -124,5 +101,5 @@
   <joint name="finger_to_ball_center" type="fixed">
     <parent link="root_finger"/>
-    <origin xyz="${finger_ball_center_xyz}" rpy="0 0 0"/>
+    <origin xyz="${finger_ball_center_xyz}" rpy="${pi/2} ${-pi/2} 0"/>
     <child link="finger_ball_center"/>
   </joint>

File: irb120_control/urdf/sensor_and_adapter_assembly.urdf (robot description, URDF)
Before this commit: robot sensor_and_adapter_assembly, 5 links, 4 joints
Links:
- link sensor_body: geometry collision mesh filename=package://irb120_control/meshes/sensor_and_adapter_assembly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 scale=1 1 1; visual mesh filename=package://irb120_control/meshes/sensor_and_adapter_assembly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 scale=1 1 1

File: irb120_moveit_config/config/irb120_macro.srdf.xacro (robot description, xacro)
@@ -30,4 +30,5 @@
     <disable_collisions link1="adapter_robot" link2="adapter_sensor" reason="Adjacent"/>
     <disable_collisions link1="adapter_sensor" link2="sensor_plate" reason="Adjacent"/>
+    <disable_collisions link1="sensor_body" link2="sensor_plate" reason="Adjacent"/>
     <disable_collisions link1="sensor_body" link2="pusher_body" reason="Adjacent"/>
     <disable_collisions link1="pusher_body" link2="ball" reason="Adjacent"/>
