Commit message: Add Realsense calibration configuration for hand-eye setup
This commit introduces a new YAML configuration file for the Realsense driver parameters specifically tailored for hand-eye calibration. The configuration optimizes the color stream settings and disables depth processing to enhance USB bandwidth utilization. The settings ensure compatibility with various resolutions while maintaining calibration accuracy.

File: irb120_control/urdf/irb120_with_finger.xacro (robot description, xacro)
@@ -10,4 +10,5 @@
   <xacro:arg name="egm_port" default="6511"/>
   <xacro:arg name="configure_via_rws" default="true"/>
+  <xacro:arg name="use_charuco_mount" default="false"/>
   <xacro:property name="prefix" value="$(arg prefix)"/>
   <xacro:property name="use_fake_hardware" value="$(arg use_fake_hardware)"/>
@@ -19,4 +20,5 @@
   <xacro:property name="egm_port" value="$(arg egm_port)"/>
   <xacro:property name="configure_via_rws" value="$(arg configure_via_rws)"/>
+  <xacro:property name="use_charuco_mount" value="$(arg use_charuco_mount)"/>
   <xacro:include filename="$(find irb120_control)/urdf/irb120_3_58_macro.xacro"/>
   <xacro:include filename="$(find irb120_control)/urdf/irb120_3_58.ros2_control.xacro"/>
@@ -34,5 +36,5 @@
     configure_via_rws="${configure_via_rws}"/>
   <!-- ====== Params to tweak ====== -->
-  <xacro:property name="ft_body_length_xyz" value="0 0 -0.02975"/>  <!-- Literallly just the sensor body length. Sensor body 'origin' is its robot-side face. -->
+  <xacro:property name="ft_body_length_xyz" value="0 0 -0.0333244"/>  <!-- Literallly just the sensor body length. Sensor body 'origin' is its robot-side face. -->
   <xacro:property name="finger_mass" value="0.066"/>           <!-- kg (measured finger+ball+screws) -->
   <xacro:property name="finger_cog" value="0.0275"/>         <!-- meters in finger frame (measured) -->
@@ -81,9 +83,20 @@
     </collision>
   </link>
-  <!-- ====== FT sensor + adapter stack, mounted to tool0 + finger and ball ====== -->
+  <!-- ====== Keep-out wall on the robot's +y side (camera stand) ====== -->
+  <!-- Collision-only (no visual), so MoveIt plans around it without it cluttering RViz.
+       Its robot-facing surface is the x-z plane at y = wall_y. -->
+  <xacro:property name="wall_y" value="0.375"/>
+  <xacro:property name="wall_thickness" value="0.05"/>
+  <xacro:property name="wall_height" value="1.2"/>
+  <link name="keepout_wall_left">
+    <collision>
+      <origin xyz="0 ${wall_thickness / 2} ${wall_height / 2}" rpy="0 0 0"/>
+      <geometry>
+        <box size="2.0 ${wall_thickness} ${wall_height}"/>
+      </geometry>
+    </collision>
+  </link>
+  <!-- The physical calibration and production chains share the robot adapters and NetFT. -->
   <xacro:include filename="$(find irb120_control)/urdf/sensor_and_adapter_assembly.urdf"/>
-  <xacro:include filename="$(find irb120_control)/urdf/finger_assembly.urdf"/>
-  <!-- ==================================== JOINTS ==================================== -->
-  <!-- connect tool0 to the Onshape assembly's root mate connector -->
   <joint name="tool0_to_sensor_root" type="fixed">
     <parent link="tool0"/>
@@ -91,17 +104,32 @@
     <child link="root_sensor"/>
   </joint>
-  <!-- connect sensor_body to finger_link (sensor body origin is its robot-side face) -->
-  <joint name="sensor_body_to_finger_root" type="fixed">
-    <parent link="sensor_body"/>
-    <origin xyz="${ft_body_length_xyz}" rpy="0 ${pi} 0"/> <!--0.3971356 ${pi/2} -1.1736581"-->
-    <child link="root_finger"/>
-  </joint>
-  <!-- finger_ball_center for EE pose (like mujoco 'site') -->
-  <link name="finger_ball_center"/>
-  <joint name="finger_to_ball_center" type="fixed">
-    <parent link="root_finger"/>
-    <origin xyz="${finger_ball_center_xyz}" rpy="${pi/2} ${-pi/2} 0"/>
-    <child link="finger_ball_center"/>
-  </joint>
+  <xacro:if value="${use_charuco_mount}">
+    <!-- Calibration-only terminal attachment. Its mounting plane is the NetFT output face. -->
+    <link name="charuco_mount">
+      <visual>
+        <geometry><mesh filename="package://irb120_control/meshes/aruco_mount.stl"/></geometry>
+        <material name="CharucoMount"><color rgba="0.95 0.55 0.05 1.0"/></material>
+      </visual>
+      <collision><geometry><mesh filename="package://irb120_control/meshes/aruco_mount.stl"/></geometry></collision>
+    </link>
+    <joint name="sensor_body_to_charuco_mount" type="fixed">
+      <parent link="sensor_body"/><child link="charuco_mount"/>
+      <origin xyz="${ft_body_length_xyz}" rpy="0 ${pi} -0.7853975"/>
+    </joint>
+  </xacro:if>
+  <xacro:unless value="${use_charuco_mount}">
+    <xacro:include filename="$(find irb120_control)/urdf/finger_assembly.urdf"/>
+    <joint name="sensor_body_to_finger_root" type="fixed">
+      <parent link="sensor_body"/>
+      <origin xyz="${ft_body_length_xyz}" rpy="0 ${pi} -0.7853975"/>
+      <child link="root_finger"/>
+    </joint>
+    <link name="finger_ball_center"/>
+    <joint name="finger_to_ball_center" type="fixed">
+      <parent link="root_finger"/>
+      <origin xyz="${finger_ball_center_xyz}" rpy="${pi/2} ${-pi/2} 0"/>
+      <child link="finger_ball_center"/>
+    </joint>
+  </xacro:unless>
   <!-- World and table should coincide, at the top table surface -->
   <joint name="world_to_table" type="fixed">
@@ -115,4 +143,10 @@
     <child link="bracket"/>
   </joint>
+  <!-- Spans the table's length (same x center), standing on the table top -->
+  <joint name="world_to_keepout_wall_left" type="fixed">
+    <parent link="world"/>
+    <origin xyz="${table_center_xyz.split()[0]} ${wall_y} 0" rpy="0 0 0"/>
+    <child link="keepout_wall_left"/>
+  </joint>
   <joint name="world_to_base" type="fixed">
     <parent link="world"/>

File: irb120_control/urdf/sensor_and_adapter_assembly.urdf (robot description, URDF)
Before this commit: robot sensor_and_adapter_assembly, 5 links, 4 joints
Links:
- link adapter_robot: geometry visual mesh filename=package://irb120_control/meshes/sensor_and_adapter_assembly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 scale=1 1 1
- link adapter_sensor: geometry visual mesh filename=package://irb120_control/meshes/sensor_and_adapter_assembly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 scale=1 1 1
- link sensor_body: mass 0.359612 -> 0.000124527; geometry visual mesh filename=package://irb120_control/meshes/sensor_and_adapter_assembly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 scale=1 1 1
- link sensor_plate: geometry visual mesh filename=package://irb120_control/meshes/sensor_and_adapter_assembly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 scale=1 1 1
Joints:
- joint fastened_1: origin xyz=0 0 0 rpy=-1.5708 0 3.14159 -> xyz=0 0 0 rpy=-1.5708 -0 3.14159
- joint fastened_2: origin xyz=0 0 0.01 rpy=3.14159 0 0 -> xyz=0 2.88889e-34 0.01 rpy=3.14159 -0 0
- joint fastened_3: origin xyz=0 0 -0.0215 rpy=0 0 0 -> xyz=6.55487e-18 1.0842e-19 -0.0215 rpy=0 -0 5.05364e-31
- joint fastened_4: origin xyz=0 0 -0.021 rpy=0 0 3.14159 -> xyz=-6.62085e-18 -0.000500516 -0.021 rpy=0 0 -2.3561975

File: irb120_moveit_config/config/irb120.srdf.xacro (robot description, xacro)
@@ -1,5 +1,13 @@
 <?xml version="1.0" encoding="utf-8"?>
 <robot xmlns:xacro="http://wiki.ros.org/xacro" name="abb_irb120_3_58">
+  <xacro:arg name="use_charuco_mount" default="false"/>
+  <xacro:property name="use_charuco_mount" value="$(arg use_charuco_mount)"/>
   <xacro:include filename="$(find irb120_moveit_config)/config/irb120_macro.srdf.xacro"/>
-  <xacro:irb120_srdf/>
+  <xacro:include filename="$(find irb120_moveit_config)/config/irb120_handeye_macro.srdf.xacro"/>
+  <xacro:if value="${use_charuco_mount}">
+    <xacro:irb120_handeye_srdf/>
+  </xacro:if>
+  <xacro:unless value="${use_charuco_mount}">
+    <xacro:irb120_srdf/>
+  </xacro:unless>
 </robot>

File: irb120_moveit_config/config/irb120_handeye_macro.srdf.xacro (robot description, xacro)
@@ -14,4 +14,7 @@
     </group_state>
     <virtual_joint name="world_joint" type="fixed" parent_frame="world" child_link="base_link"/>
+    <!-- The keep-out wall is fixed to the world and overlaps the table/bracket edges by design. -->
+    <disable_collisions link1="keepout_wall_left" link2="table" reason="Adjacent"/>
+    <disable_collisions link1="keepout_wall_left" link2="bracket" reason="Adjacent"/>
     <disable_collisions link1="base_link" link2="link_1" reason="Adjacent"/>
     <disable_collisions link1="link_1" link2="link_2" reason="Adjacent"/>
@@ -25,6 +28,10 @@
     <disable_collisions link1="link_4" link2="link_6" reason="Never"/>
     <disable_collisions link1="link_5" link2="link_6" reason="Adjacent"/>
-    <disable_collisions link1="link_6" link2="ft_link" reason="Adjacent"/>
-    <disable_collisions link1="ft_link" link2="finger_link" reason="Adjacent"/>
+    <disable_collisions link1="link_6" link2="adapter_robot" reason="Adjacent"/>
+    <disable_collisions link1="link_6" link2="adapter_sensor" reason="Adjacent"/>
+    <disable_collisions link1="adapter_robot" link2="adapter_sensor" reason="Adjacent"/>
+    <disable_collisions link1="adapter_sensor" link2="sensor_plate" reason="Adjacent"/>
+    <disable_collisions link1="sensor_plate" link2="sensor_body" reason="Adjacent"/>
+    <disable_collisions link1="sensor_body" link2="charuco_mount" reason="Adjacent"/>
   </xacro:macro>
 </robot>

File: irb120_moveit_config/config/irb120_macro.srdf.xacro (robot description, xacro)
@@ -14,4 +14,7 @@
     </group_state>
     <virtual_joint name="world_joint" type="fixed" parent_frame="world" child_link="base_link"/>
+    <!-- The keep-out wall is fixed to the world and overlaps the table/bracket edges by design. -->
+    <disable_collisions link1="keepout_wall_left" link2="table" reason="Adjacent"/>
+    <disable_collisions link1="keepout_wall_left" link2="bracket" reason="Adjacent"/>
     <disable_collisions link1="base_link" link2="link_1" reason="Adjacent"/>
     <disable_collisions link1="link_1" link2="link_2" reason="Adjacent"/>

Commit message: Enhance object handling in motion planning by introducing object_obstacle context manager for collision avoidance. Update related functions to utilize the detected object cloud for safer approach and return maneuvers. Adjust standoff distances for improved clearance during pushes and squashes. Document changes in README and add new engineering notes for push test findings.

File: irb120_control/urdf/irb120_with_finger.xacro (robot description, xacro)
@@ -104,4 +104,19 @@
     <child link="root_sensor"/>
   </joint>
+  <!-- The adapters, sensor plate and NetFT body have no collision geometry of their own; one
+       oversized cylinder covers all of them: 90 mm diameter, from the tool0 flange face to the
+       sensor's output face where the finger / ChArUco mount attaches (85.8 mm along tool0 +X). -->
+  <xacro:property name="tool_stack_length" value="0.0858"/>
+  <link name="tool_stack_collision">
+    <collision>
+      <origin xyz="${tool_stack_length / 2} 0 0" rpy="0 ${pi/2} 0"/>
+      <geometry><cylinder radius="0.045" length="${tool_stack_length}"/></geometry>
+    </collision>
+  </link>
+  <joint name="tool0_to_tool_stack_collision" type="fixed">
+    <parent link="tool0"/>
+    <origin xyz="0 0 0" rpy="0 0 0"/>
+    <child link="tool_stack_collision"/>
+  </joint>
   <xacro:if value="${use_charuco_mount}">
     <!-- Calibration-only terminal attachment. Its mounting plane is the NetFT output face. -->

File: irb120_moveit_config/config/irb120_handeye_macro.srdf.xacro (robot description, xacro)
@@ -29,4 +29,7 @@
     <disable_collisions link1="link_5" link2="link_6" reason="Adjacent"/>
     <disable_collisions link1="link_6" link2="adapter_robot" reason="Adjacent"/>
+    <disable_collisions link1="link_5" link2="tool_stack_collision" reason="Adjacent"/> <!-- tool-stack cylinder, see irb120_with_finger.xacro -->
+    <disable_collisions link1="link_6" link2="tool_stack_collision" reason="Adjacent"/>
+    <disable_collisions link1="tool_stack_collision" link2="charuco_mount" reason="Adjacent"/>
     <disable_collisions link1="link_6" link2="adapter_sensor" reason="Adjacent"/>
     <disable_collisions link1="adapter_robot" link2="adapter_sensor" reason="Adjacent"/>

File: irb120_moveit_config/config/irb120_macro.srdf.xacro (robot description, xacro)
@@ -30,4 +30,7 @@
     <disable_collisions link1="link_5" link2="adapter_sensor" reason="Adjacent"/> <!-- Recall the adapter 'sticks into' the tool0 to be secure. This avoids collision.-->
     <disable_collisions link1="link_6" link2="adapter_robot" reason="Adjacent"/>
+    <disable_collisions link1="link_5" link2="tool_stack_collision" reason="Adjacent"/> <!-- tool-stack cylinder, see irb120_with_finger.xacro -->
+    <disable_collisions link1="link_6" link2="tool_stack_collision" reason="Adjacent"/>
+    <disable_collisions link1="tool_stack_collision" link2="pusher_body" reason="Adjacent"/>
     <disable_collisions link1="link_6" link2="adapter_sensor" reason="Adjacent"/>
     <disable_collisions link1="adapter_robot" link2="adapter_sensor" reason="Adjacent"/>
