Commit message: Added new calibration script and ran it plus added taring before each press motion.

File: irb120_models/urdf/finger_assembly.urdf (robot description, URDF)
Before this commit: robot finger_assembly, 3 links, 2 joints
Links:
- link ball: geometry collision mesh filename=package://irb120_models/meshes/finger_assembly/ball.gltf scale=1 1 1; visual mesh filename=package://irb120_models/meshes/finger_assembly/ball.gltf scale=1 1 1
- link pusher_body: geometry collision mesh filename=package://irb120_models/meshes/finger_assembly/pusher_body.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 scale=1 1 1; visual mesh filename=package://irb120_models/meshes/finger_assembly/pusher_body.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 scale=1 1 1

File: irb120_models/urdf/irb120_3_58.xacro (robot description, xacro)
@@ -17,6 +17,6 @@
   <xacro:property name="egm_port" value="$(arg egm_port)"/>
   <xacro:property name="configure_via_rws" value="$(arg configure_via_rws)"/>
-  <xacro:include filename="$(find irb120_control)/urdf/irb120_3_58_macro.xacro"/>
-  <xacro:include filename="$(find irb120_control)/urdf/irb120_3_58.ros2_control.xacro"/>
+  <xacro:include filename="$(find irb120_models)/urdf/irb120_3_58_macro.xacro"/>
+  <xacro:include filename="$(find irb120_models)/urdf/irb120_3_58.ros2_control.xacro"/>
   <xacro:abb_irb120_3_58 prefix=""/>
   <xacro:abb_irb120_3_58_ros2_control

File: irb120_models/urdf/irb120_3_58_macro.xacro (robot description, xacro)
@@ -13,12 +13,12 @@
         <origin xyz="0 0 0" rpy="0 0 0"/>
         <geometry>
-          <mesh filename="package://irb120_control/meshes/irb120_3_58/visual/base_link.stl"/>
-        </geometry>
-        <xacro:material_abb_orange />
-      </visual>
-      <collision>
-        <origin xyz="0 0 0" rpy="0 0 0"/>
-        <geometry>
-          <mesh filename="package://irb120_control/meshes/irb120_3_58/collision/base_link.stl"/>
+          <mesh filename="package://irb120_models/meshes/irb120_3_58/visual/base_link.stl"/>
+        </geometry>
+        <xacro:material_abb_orange />
+      </visual>
+      <collision>
+        <origin xyz="0 0 0" rpy="0 0 0"/>
+        <geometry>
+          <mesh filename="package://irb120_models/meshes/irb120_3_58/collision/base_link.stl"/>
         </geometry>
         <xacro:material_abb_yellow />
@@ -34,12 +34,12 @@
         <origin xyz="0 0 0" rpy="0 0 0"/>
         <geometry>
-          <mesh filename="package://irb120_control/meshes/irb120_3_58/visual/link_1.stl"/>
-        </geometry>
-        <xacro:material_abb_orange />
-      </visual>
-      <collision>
-        <origin xyz="0 0 0" rpy="0 0 0"/>
-        <geometry>
-          <mesh filename="package://irb120_control/meshes/irb120_3_58/collision/link_1.stl"/>
+          <mesh filename="package://irb120_models/meshes/irb120_3_58/visual/link_1.stl"/>
+        </geometry>
+        <xacro:material_abb_orange />
+      </visual>
+      <collision>
+        <origin xyz="0 0 0" rpy="0 0 0"/>
+        <geometry>
+          <mesh filename="package://irb120_models/meshes/irb120_3_58/collision/link_1.stl"/>
         </geometry>
         <xacro:material_abb_yellow />
@@ -55,12 +55,12 @@
         <origin xyz="0 0 0" rpy="0 0 0"/>
         <geometry>
-          <mesh filename="package://irb120_control/meshes/irb120_3_58/visual/link_2.stl"/>
-        </geometry>
-        <xacro:material_abb_orange />
-      </visual>
-      <collision>
-        <origin xyz="0 0 0" rpy="0 0 0"/>
-        <geometry>
-          <mesh filename="package://irb120_control/meshes/irb120_3_58/collision/link_2.stl"/>
+          <mesh filename="package://irb120_models/meshes/irb120_3_58/visual/link_2.stl"/>
+        </geometry>
+        <xacro:material_abb_orange />
+      </visual>
+      <collision>
+        <origin xyz="0 0 0" rpy="0 0 0"/>
+        <geometry>
+          <mesh filename="package://irb120_models/meshes/irb120_3_58/collision/link_2.stl"/>
         </geometry>
         <xacro:material_abb_yellow />
@@ -76,12 +76,12 @@
         <origin xyz="0 0 0" rpy="0 0 0"/>
         <geometry>
-          <mesh filename="package://irb120_control/meshes/irb120_3_58/visual/link_3.stl"/>
-        </geometry>
-        <xacro:material_abb_orange />
-      </visual>
-      <collision>
-        <origin xyz="0 0 0" rpy="0 0 0"/>
-        <geometry>
-          <mesh filename="package://irb120_control/meshes/irb120_3_58/collision/link_3.stl"/>
+          <mesh filename="package://irb120_models/meshes/irb120_3_58/visual/link_3.stl"/>
+        </geometry>
+        <xacro:material_abb_orange />
+      </visual>
+      <collision>
+        <origin xyz="0 0 0" rpy="0 0 0"/>
+        <geometry>
+          <mesh filename="package://irb120_models/meshes/irb120_3_58/collision/link_3.stl"/>
         </geometry>
         <xacro:material_abb_yellow />
@@ -97,12 +97,12 @@
         <origin xyz="0 0 0" rpy="0 0 0"/>
         <geometry>
-          <mesh filename="package://irb120_control/meshes/irb120_3_58/visual/link_4.stl"/>
-        </geometry>
-        <xacro:material_abb_orange />
-      </visual>
-      <collision>
-        <origin xyz="0 0 0" rpy="0 0 0"/>
-        <geometry>
-          <mesh filename="package://irb120_control/meshes/irb120_3_58/collision/link_4.stl"/>
+          <mesh filename="package://irb120_models/meshes/irb120_3_58/visual/link_4.stl"/>
+        </geometry>
+        <xacro:material_abb_orange />
+      </visual>
+      <collision>
+        <origin xyz="0 0 0" rpy="0 0 0"/>
+        <geometry>
+          <mesh filename="package://irb120_models/meshes/irb120_3_58/collision/link_4.stl"/>
         </geometry>
         <xacro:material_abb_yellow />
@@ -118,12 +118,12 @@
         <origin xyz="0 0 0" rpy="0 0 0"/>
         <geometry>
-          <mesh filename="package://irb120_control/meshes/irb120_3_58/visual/link_5.stl"/>
-        </geometry>
-        <xacro:material_abb_orange />
-      </visual>
-      <collision>
-        <origin xyz="0 0 0" rpy="0 0 0"/>
-        <geometry>
-          <mesh filename="package://irb120_control/meshes/irb120_3_58/collision/link_5.stl"/>
+          <mesh filename="package://irb120_models/meshes/irb120_3_58/visual/link_5.stl"/>
+        </geometry>
+        <xacro:material_abb_orange />
+      </visual>
+      <collision>
+        <origin xyz="0 0 0" rpy="0 0 0"/>
+        <geometry>
+          <mesh filename="package://irb120_models/meshes/irb120_3_58/collision/link_5.stl"/>
         </geometry>
         <xacro:material_abb_yellow />
@@ -139,5 +139,5 @@
         <origin xyz="0 0 0" rpy="0 0 0"/>
         <geometry>
-          <mesh filename="package://irb120_control/meshes/irb120_3_58/visual/link_6.stl"/>
+          <mesh filename="package://irb120_models/meshes/irb120_3_58/visual/link_6.stl"/>
         </geometry>
         <xacro:material_abb_black />
@@ -146,5 +146,5 @@
         <origin xyz="0 0 0" rpy="0 0 0"/>
         <geometry>
-          <mesh filename="package://irb120_control/meshes/irb120_3_58/collision/link_6.stl"/>
+          <mesh filename="package://irb120_models/meshes/irb120_3_58/collision/link_6.stl"/>
         </geometry>
         <xacro:material_abb_yellow />

File: irb120_models/urdf/irb120_with_finger.xacro (robot description, xacro)
@@ -21,6 +21,6 @@
   <xacro:property name="configure_via_rws" value="$(arg configure_via_rws)"/>
   <xacro:property name="use_charuco_mount" value="$(arg use_charuco_mount)"/>
-  <xacro:include filename="$(find irb120_control)/urdf/irb120_3_58_macro.xacro"/>
-  <xacro:include filename="$(find irb120_control)/urdf/irb120_3_58.ros2_control.xacro"/>
+  <xacro:include filename="$(find irb120_models)/urdf/irb120_3_58_macro.xacro"/>
+  <xacro:include filename="$(find irb120_models)/urdf/irb120_3_58.ros2_control.xacro"/>
   <xacro:abb_irb120_3_58 prefix="${prefix}"/>
   <xacro:abb_irb120_3_58_ros2_control
@@ -98,5 +98,5 @@
   </link>
   <!-- The physical calibration and production chains share the robot adapters and NetFT. -->
-  <xacro:include filename="$(find irb120_control)/urdf/sensor_and_adapter_assembly.urdf"/>
+  <xacro:include filename="$(find irb120_models)/urdf/sensor_and_adapter_assembly.urdf"/>
   <joint name="tool0_to_sensor_root" type="fixed">
     <parent link="tool0"/>
@@ -123,8 +123,8 @@
     <link name="charuco_mount">
       <visual>
-        <geometry><mesh filename="package://irb120_control/meshes/aruco_mount.stl"/></geometry>
+        <geometry><mesh filename="package://irb120_models/meshes/aruco_mount.stl"/></geometry>
         <material name="CharucoMount"><color rgba="0.95 0.55 0.05 1.0"/></material>
       </visual>
-      <collision><geometry><mesh filename="package://irb120_control/meshes/aruco_mount.stl"/></geometry></collision>
+      <collision><geometry><mesh filename="package://irb120_models/meshes/aruco_mount.stl"/></geometry></collision>
     </link>
     <joint name="sensor_body_to_charuco_mount" type="fixed">
@@ -134,5 +134,5 @@
   </xacro:if>
   <xacro:unless value="${use_charuco_mount}">
-    <xacro:include filename="$(find irb120_control)/urdf/finger_assembly.urdf"/>
+    <xacro:include filename="$(find irb120_models)/urdf/finger_assembly.urdf"/>
     <joint name="sensor_body_to_finger_root" type="fixed">
       <parent link="sensor_body"/>

File: irb120_models/urdf/sensor_and_adapter_assembly.urdf (robot description, URDF)
Before this commit: robot sensor_and_adapter_assembly, 5 links, 4 joints
Links:
- link adapter_robot: geometry visual mesh filename=package://irb120_models/meshes/sensor_and_adapter_assembly/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 scale=1 1 1
- link adapter_sensor: geometry visual mesh filename=package://irb120_models/meshes/sensor_and_adapter_assembly/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 scale=1 1 1
- link sensor_body: geometry visual mesh filename=package://irb120_models/meshes/sensor_and_adapter_assembly/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 scale=1 1 1
- link sensor_plate: geometry visual mesh filename=package://irb120_models/meshes/sensor_and_adapter_assembly/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 scale=1 1 1
